File: hardware/development_board/devboard_v2/kicad/1_01POWER.kicad_sch (KiCad schematic)
At the start: 79 parts, among them IC2 SY8088IAAC, J6 1982633-1, J8 U6252-35c, M1 TP, Q4 RE1C001ZPTL, Q5 RE1C001UNTCL, Q6 RE1C001ZPTL, Q7 RE1C001ZPTL, Q8 BSS123-TP, Q9 RE1C001UNTCL, SW13 TS-1095PS-A1B2-C3D2, SW14 TP, U1 MP2607DL-LF-P, U2 XC6194AA05ER-G, U3 NCP115AMX150TCG, U8 NCP115AMX180TCG, U9 NCP115AMX280TCG

Commit message: Rename devboard v2 files to remove spaces from paths.
Replace spaces with underscores in KiCad, gerber, and footprint filenames so the branch can be committed and pushed on GitHub without path issues.
Parts:
- 1V5, 1V8, 2V8, GND1, SC_SW1, SW14, V3P0, VBAT1, VIN1, VSW1, VSYS1: footprint ProPrj_Seg-easyedapro:TESTPOINT 1MM -> ProPrj_Seg-easyedapro:TESTPOINT_1MM; Origin Footprint TESTPOINT 1MM -> TESTPOINT_1MM
- B1: footprint ProPrj_Seg-easyedapro:PLAGE - ROUGE -> ProPrj_Seg-easyedapro:PLAGE_-_ROUGE; Origin Footprint PLAGE - ROUGE -> PLAGE_-_ROUGE
- D2: footprint ProPrj_Seg-easyedapro:OSRAM LRY8SFU1V21 -> ProPrj_Seg-easyedapro:OSRAM_LRY8SFU1V21; Origin Footprint OSRAM LRY8SFU1V21 -> OSRAM_LRY8SFU1V21
- F1, F2: footprint ProPrj_Seg-easyedapro:0805 - FUSE -> ProPrj_Seg-easyedapro:0805_-_FUSE; Origin Footprint 0805 - FUSE -> 0805_-_FUSE
- IC2: footprint ProPrj_Seg-easyedapro:SOT23-5 0.95 VAR AA -> ProPrj_Seg-easyedapro:SOT23-5_0.95_VAR_AA
- J6: footprint ProPrj_Seg-easyedapro:TE 19826331 -> ProPrj_Seg-easyedapro:TE_19826331; Origin Footprint TE 19826331 -> TE_19826331
- J8: footprint ProPrj_Seg-easyedapro:ANTENK U6252-35C -> ProPrj_Seg-easyedapro:ANTENK_U6252-35C; Origin Footprint ANTENK U6252-35C -> ANTENK_U6252-35C
- M1: footprint ProPrj_Seg-easyedapro:PLAGE - NOIRE -> ProPrj_Seg-easyedapro:PLAGE_-_NOIRE; Origin Footprint PLAGE - NOIRE -> PLAGE_-_NOIRE
- U2: footprint ProPrj_Seg-easyedapro:TOREX USP-8B06 -> ProPrj_Seg-easyedapro:TOREX_USP-8B06; Origin Footprint TOREX USP-8B06 -> TOREX_USP-8B06
- U3, U8, U9: footprint ProPrj_Seg-easyedapro:ON SEMI NCV8160AMX330TBG -> ProPrj_Seg-easyedapro:ON_SEMI_NCV8160AMX330TBG; Origin Footprint ON SEMI NCV8160AMX330TBG -> ON_SEMI_NCV8160AMX330TBG
