File: hardware/development_board/devboard_v2/kicad/2_02MCU.kicad_sch (KiCad schematic)
At the start: 44 parts, among them CN1 HX JN1.27-2x10 TP H4.9, J1V8 TP, P210 TC2030-MCP-NL, U11 Sort_Symbol, U12 STM32H573VIT6, U13 Sort_Symbol, U14 Sort_Symbol, U15 Sort_Symbol, U4 Sort_Symbol, U5 TLVH431AQDBZRG4, U6 Sort_Symbol

Commit message: Rename devboard v2 files to remove spaces from paths.
Replace spaces with underscores in KiCad, gerber, and footprint filenames so the branch can be committed and pushed on GitHub without path issues.
Parts:
- GND4, J1V8, JGND1, JRST1, JSWC1, JSWD1, JTDI1, JTDO1, Rx4, Tx4: footprint ProPrj_Seg-easyedapro:TESTPOINT 1MM -> ProPrj_Seg-easyedapro:TESTPOINT_1MM; Origin Footprint TESTPOINT 1MM -> TESTPOINT_1MM
Changed lines of the file:
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@@
 			)
 		)
-		(property "Footprint" "ProPrj_Seg-easyedapro:TESTPOINT 1MM"
+		(property "Footprint" "ProPrj_Seg-easyedapro:TESTPOINT_1MM"
 			(at 294.64 161.29 0)
 			(effects
@@
 			)
 		)
-		(property "Origin Footprint" "TESTPOINT 1MM"
+		(property "Origin Footprint" "TESTPOINT_1MM"
 			(at 294.64 161.29 0)
 			(effects
@@
 			)
 		)
-		(property "Footprint" "ProPrj_Seg-easyedapro:TESTPOINT 1MM"
+		(property "Footprint" "ProPrj_Seg-easyedapro:TESTPOINT_1MM"
 			(at 219.71 62.23 0)
 			(effects
@@
 			)
 		)
-		(property "Origin Footprint" "TESTPOINT 1MM"
+		(property "Origin Footprint" "TESTPOINT_1MM"
 			(at 219.71 62.23 0)
 			(effects
@@
 			)
 		)
-		(property "Footprint" "ProPrj_Seg-easyedapro:TESTPOINT 1MM"
+		(property "Footprint" "ProPrj_Seg-easyedapro:TESTPOINT_1MM"
 			(at 294.64 158.75 0)
 			(effects
@@
 			)
 		)
-		(property "Origin Footprint" "TESTPOINT 1MM"
+		(property "Origin Footprint" "TESTPOINT_1MM"
 			(at 294.64 158.75 0)
 			(effects
@@
 			)
 		)
-		(property "Footprint" "ProPrj_Seg-easyedapro:TESTPOINT 1MM"
+		(property "Footprint" "ProPrj_Seg-easyedapro:TESTPOINT_1MM"
 			(at 294.64 163.83 0)
 			(effects
@@
 			)
 		)
-		(property "Origin Footprint" "TESTPOINT 1MM"
+		(property "Origin Footprint" "TESTPOINT_1MM"
 			(at 294.64 163.83 0)
 			(effects
@@
 			)
 		)
-		(property "Footprint" "ProPrj_Seg-easyedapro:TESTPOINT 1MM"
+		(property "Footprint" "ProPrj_Seg-easyedapro:TESTPOINT_1MM"
 			(at 121.92 109.22 0)
 			(effects
@@
 			)
 		)
-		(property "Origin Footprint" "TESTPOINT 1MM"
+		(property "Origin Footprint" "TESTPOINT_1MM"
 			(at 120.65 115.57 90)
 			(effects
@@
 			)
 		)
-		(property "Footprint" "ProPrj_Seg-easyedapro:TESTPOINT 1MM"
+		(property "Footprint" "ProPrj_Seg-easyedapro:TESTPOINT_1MM"
 			(at 294.64 156.21 0)
 			(effects
@@
 			)
 		)
-		(property "Origin Footprint" "TESTPOINT 1MM"
+		(property "Origin Footprint" "TESTPOINT_1MM"
 			(at 294.64 156.21 0)
 			(effects
@@
 			)
 		)
-		(property "Footprint" "ProPrj_Seg-easyedapro:TESTPOINT 1MM"
+		(property "Footprint" "ProPrj_Seg-easyedapro:TESTPOINT_1MM"
 			(at 294.64 166.37 0)
 			(effects
@@
 			)
 		)
-		(property "Origin Footprint" "TESTPOINT 1MM"
+		(property "Origin Footprint" "TESTPOINT_1MM"
 			(at 294.64 166.37 0)
 			(effects
@@
 			)
 		)
-		(property "Footprint" "ProPrj_Seg-easyedapro:TESTPOINT 1MM"
+		(property "Footprint" "ProPrj_Seg-easyedapro:TESTPOINT_1MM"
 			(at 121.92 106.68 0)
 			(effects
@@
 			)
 		)
-		(property "Origin Footprint" "TESTPOINT 1MM"
+		(property "Origin Footprint" "TESTPOINT_1MM"
 			(at 120.65 113.03 90)
 			(effects
@@
 			)
 		)
-		(property "Footprint" "ProPrj_Seg-easyedapro:TESTPOINT 1MM"
+		(property "Footprint" "ProPrj_Seg-easyedapro:TESTPOINT_1MM"
 			(at 294.64 168.91 0)
 			(effects
@@
 			)
 		)
-		(property "Origin Footprint" "TESTPOINT 1MM"
+		(property "Origin Footprint" "TESTPOINT_1MM"
 			(at 294.64 168.91 0)
 			(effects
@@
 			)
 		)
-		(property "Footprint" "ProPrj_Seg-easyedapro:TESTPOINT 1MM"
+		(property "Footprint" "ProPrj_Seg-easyedapro:TESTPOINT_1MM"
 			(at 294.64 171.45 0)
 			(effects
@@
 			)
 		)
-		(property "Origin Footprint" "TESTPOINT 1MM"
+		(property "Origin Footprint" "TESTPOINT_1MM"
 			(at 294.64 171.45 0)
 			(effects
