File: hardware/development_board/devboard_v2/kicad/3_03PERIPHERALS.kicad_sch (KiCad schematic)
At the start: 33 parts, among them J2 FFC2B35-12-G, Q3 RZM002P02T2L, SW1 TS-1095PS-A1B2-C3D2, SW10 TS-1095PS-A1B2-C3D2, SW11 TS-1095PS-A1B2-C3D2, SW12 TS-1095PS-A1B2-C3D2, SW2 TS-1095PS-A1B2-C3D2, SW3 TS-1095PS-A1B2-C3D2, SW4 TS-1095PS-A1B2-C3D2, SW5 TS-1095PS-A1B2-C3D2, SW6 TS-1095PS-A1B2-C3D2, SW7 TS-1095PS-A1B2-C3D2, SW8 TS-1095PS-A1B2-C3D2, SW9 TS-1095PS-A1B2-C3D2, T1 NTR3C21NZT1G, U7 ESDS312DBVR, X1 HC-FPC-05-09-24RLTAG

Commit message: Rename devboard v2 files to remove spaces from paths.
Replace spaces with underscores in KiCad, gerber, and footprint filenames so the branch can be committed and pushed on GitHub without path issues.
Parts:
- J2: footprint ProPrj_Seg-easyedapro:GCT FFC2B35-12-G -> ProPrj_Seg-easyedapro:GCT_FFC2B35-12-G; Origin Footprint GCT FFC2B35-12-G -> GCT_FFC2B35-12-G
- R12: footprint ProPrj_Seg-easyedapro:0402 - RESISTOR -> ProPrj_Seg-easyedapro:0402_-_RESISTOR; Origin Footprint 0402 - RESISTOR -> 0402_-_RESISTOR
- X1: footprint ProPrj_Seg-easyedapro:HCTL HC-FPC-05-09-24RLTAG -> ProPrj_Seg-easyedapro:HCTL_HC-FPC-05-09-24RLTAG; symbol ProPrj_Seg-easyedapro:HCTL HC-FPC-05-09-24RLTAG -> ProPrj_Seg-easyedapro:HCTL_HC-FPC-05-09-24RLTAG; Design Item ID HCTL HC-FPC-05-09-24RLTAG -> HCTL_HC-FPC-05-09-24RLTAG; Origin Footprint HCTL HC-FPC-05-09-24RLTAG -> HCTL_HC-FPC-05-09-24RLTAG
Changed lines of the file:
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@@
 			)
 		)
-		(property "Footprint" "ProPrj_Seg-easyedapro:GCT FFC2B35-12-G"
+		(property "Footprint" "ProPrj_Seg-easyedapro:GCT_FFC2B35-12-G"
 			(at 231.14 67.31 0)
 			(effects
@@
 			)
 		)
-		(property "Origin Footprint" "GCT FFC2B35-12-G"
+		(property "Origin Footprint" "GCT_FFC2B35-12-G"
 			(at 231.14 67.31 0)
 			(effects
@@
 	)
 	(symbol
-		(lib_id "ProPrj_Seg-easyedapro:HCTL HC-FPC-05-09-24RLTAG")
+		(lib_id "ProPrj_Seg-easyedapro:HCTL_HC-FPC-05-09-24RLTAG")
 		(at 292.1 69.85 0)
 		(unit 1)
@@
 			)
 		)
-		(property "Footprint" "ProPrj_Seg-easyedapro:HCTL HC-FPC-05-09-24RLTAG"
+		(property "Footprint" "ProPrj_Seg-easyedapro:HCTL_HC-FPC-05-09-24RLTAG"
 			(at 292.1 69.85 0)
 			(effects
@@
 			)
 		)
-		(property "Design Item ID" "HCTL HC-FPC-05-09-24RLTAG"
+		(property "Design Item ID" "HCTL_HC-FPC-05-09-24RLTAG"
 			(at 292.1 69.85 0)
 			(effects
@@
 			)
 		)
-		(property "Origin Footprint" "HCTL HC-FPC-05-09-24RLTAG"
+		(property "Origin Footprint" "HCTL_HC-FPC-05-09-24RLTAG"
 			(at 292.1 69.85 0)
 			(effects
@@
 			)
 		)
-		(property "Footprint" "ProPrj_Seg-easyedapro:0402 - RESISTOR"
+		(property "Footprint" "ProPrj_Seg-easyedapro:0402_-_RESISTOR"
 			(at 205.74 74.93 0)
 			(effects
@@
 			)
 		)
-		(property "Origin Footprint" "0402 - RESISTOR"
+		(property "Origin Footprint" "0402_-_RESISTOR"
 			(at 205.74 74.93 0)
 			(effects
